File: ice4pi.kicad_pcb (KiCad board)
At the start: 4 copper layers, 65 x 30 mm, 66 parts, among them J1 Pmod 2x6, J2 Raspberry_Pi_2_3, U1 ICE40HX1K-TQ144, U2 W25Q32JVSSIQ, U3 LT3030, U4 DSC1001DI1-012.0000, U5 TFDU4101-TR3

Commit message: Release pi-bridge-1-1
Parts:
- removed C1, C16, C20, C30, C4: 10uF, Capacitor_SMD:C_0402_1005Metric
- removed C10, C11, C13, C15, C27, C29, C5, C6: 0.01uF, Capacitor_SMD:C_0402_1005Metric
- removed C12, C14, C18, C19, C2, C21, C23, C24, C25, C26, C28, C3, C32, C9: 0.1uF, Capacitor_SMD:C_0402_1005Metric
- removed C17, C22: 1 uF, Capacitor_SMD:C_0402_1005Metric
- removed C31, C8: 4.7uF, Capacitor_SMD:C_0402_1005Metric
- removed D1, D2, D3, D4, D5: LED, LED_SMD:LED_0402_1005Metric
- removed D6: CDBU0520, Diode_SMD:D_0603_1608Metric
- removed R1: 1M, Resistor_SMD:R_0402_1005Metric
- removed R10, R11, R12, R13, R14: 1K, Resistor_SMD:R_0402_1005Metric
- removed R15, R16, R17, R18, R19, R2: 10K, Resistor_SMD:R_0402_1005Metric
- removed R20, R7: 100, Resistor_SMD:R_0402_1005Metric
- removed R21, R22: 47, Resistor_SMD:R_0402_1005Metric
- removed R9: 0.1, Resistor_SMD:R_0402_1005Metric
- removed U1: ICE40HX1K-TQ144, Package_QFP:TQFP-144_20x20mm_P0.5mm
- removed U2: W25Q32JVSSIQ, Package_SO:SOIC-8_3.9x4.9mm_P1.27mm
- removed U3: LT3030, ice4pi:TSSOP-20_4.4x6.5mm_P0.65mm
- removed U4: DSC1001DI1-012.0000, Oscillator:Oscillator_SMD_Abracon_ASDMB-4Pin_2.5x2.0mm
- removed U5: TFDU4101-TR3, ice4pi:TFDU4101-TR3
- J1: value Pmod 2x6 -> Conn_02x20_Odd_Even; footprint ice4pi:PinSocket_2x06_P2.54mm_Vertical_1to6_7to12 -> ice4pi:PinSocket_2x20_P2.54mm_Vertical_1_04mm; moved to B.Cu
- J2: value Raspberry_Pi_2_3 -> Conn_02x20_Odd_Even
- moved J1 51.3 mm to (58.4, 76.8), turned to 270 degrees
- moved svg2mod 20.0 mm to (83.0, 64.0), turned to 90 degrees
Connections:
- J1 pad 1: PIO1_02 -> +3V3
- J1 pad 10: PIO1_09 -> Net-(J1-Pad10)
- J1 pad 11: GND -> Net-(J1-Pad11)
- J1 pad 12: +3V3 -> Net-(J1-Pad12)
- J1 pad 2: PIO1_03 -> +5V
- J1 pad 3: PIO1_04 -> Net-(J1-Pad3)
- J1 pad 4: PIO1_05 -> +5V
- J1 pad 5: GND -> Net-(J1-Pad5)
- J1 pad 6: +3V3 -> GND
- J1 pad 7: PIO1_06 -> Net-(J1-Pad7)
- J1 pad 8: PIO1_07 -> Net-(J1-Pad8)
- J1 pad 9: PIO1_08 -> GND
- J2 pad 10: RS232_Tx_TTL -> Net-(J1-Pad10)
- J2 pad 11: PIO0_18 -> Net-(J1-Pad11)
- J2 pad 12: PIO0_17 -> Net-(J1-Pad12)
- J2 pad 13: PIO0_16 -> Net-(J1-Pad13)
- J2 pad 15: PIO0_14 -> Net-(J1-Pad15)
- J2 pad 16: PIO0_15 -> Net-(J1-Pad16)
- J2 pad 18: iCE_CREST -> Net-(J1-Pad18)
- J2 pad 19: iCE_MOSI -> Net-(J1-Pad19)
- J2 pad 21: iCE_MISO -> Net-(J1-Pad21)
- J2 pad 22: iCE_CDONE -> Net-(J1-Pad22)
- J2 pad 23: iCE_SCK -> Net-(J1-Pad23)
- J2 pad 24: iCE_SS_B -> Net-(J1-Pad24)
- J2 pad 26: PIO0_13 -> Net-(J1-Pad26)
- J2 pad 27: PIO0_11 -> Net-(J1-Pad27)
- J2 pad 28: PIO0_12 -> Net-(J1-Pad28)
- J2 pad 29: PIO0_10 -> Net-(J1-Pad29)
- J2 pad 3: PIO0_20 -> Net-(J1-Pad3)
- J2 pad 31: PIO0_08 -> Net-(J1-Pad31)
- J2 pad 32: PIO0_09 -> Net-(J1-Pad32)
- J2 pad 33: PIO0_07 -> Net-(J1-Pad33)
- J2 pad 35: PIO0_05 -> Net-(J1-Pad35)
- J2 pad 36: PIO0_06 -> Net-(J1-Pad36)
- J2 pad 37: PIO0_03 -> Net-(J1-Pad37)
- J2 pad 38: PIO0_04 -> Net-(J1-Pad38)
- J2 pad 40: PIO0_02 -> Net-(J1-Pad40)
- J2 pad 5: PIO0_21 -> Net-(J1-Pad5)
- J2 pad 7: PIO0_19 -> Net-(J1-Pad7)
- J2 pad 8: RS232_Rx_TTL -> Net-(J1-Pad8)
Routing:
- net iCE_MOSI: track 67.9 -> 0.00 mm, vias 2 -> 0
- net iCE_SCK: track 60.9 -> 0.00 mm, vias 3 -> 0
- net iCE_SS_B: track 58.3 -> 0.00 mm, vias 3 -> 0
- net iCE_MISO: track 57.9 -> 0.00 mm, vias 4 -> 0
- net GND: track 134.7 -> 192.5 mm, vias 35 -> 0
- net +1V2: track 46.8 -> 0.00 mm, vias 8 -> 0
- net IR_SD: track 41.6 -> 0.00 mm, vias 2 -> 0
- net iCE_CDONE: track 39.7 -> 0.00 mm, vias 1 -> 0
- net PIO0_04: track 37.6 -> 0.00 mm, vias 3 -> 0
- net iCE_CREST: track 37.1 -> 0.00 mm, vias 1 -> 0
- net PIO0_06: track 35.4 -> 0.00 mm, vias 2 -> 0
- net +3V3: track 79.6 -> 48.1 mm, vias 23 -> 0
- net PIO0_09: track 30.9 -> 0.00 mm, vias 1 -> 0
- net PIO0_05: track 30.9 -> 0.00 mm, vias 1 -> 0
- net PIO0_02: track 30.4 -> 0.00 mm, vias 1 -> 0
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- added copper zone on In2.Cu, net +5V
- removed copper zone on In2.Cu, net +1V2
- removed copper zone on In2.Cu, net +3V3
Other:
- outline, holes or cut-outs redrawn
- board text added: "^"
- board text added: "pi-bridge-1-1"
- board text removed: "ice4pi ver. 1.2"

Commit message: Release pi-bridge-2mm-1-1
Parts:
- removed the ? at (53.5, 75.5)
- removed the ? at (111.5, 75.5)
- removed the svg2mod at (83.0, 64.0)
- added ?: , ice4pi:mount_hole, F.Cu at (53.5, 63.5)
- added ?: , ice4pi:mount_hole, F.Cu at (111.5, 63.5)
- added svg2mod: G***, ice4pi:lsi-logo-32mm, F.Cu at (99.0, 59.0)
- moved J1 12.0 mm to (58.4, 64.8)
Routing:
- net GND: track 192.5 -> 96.6 mm
- net +3V3: track 48.1 -> 24.1 mm
- net +5V: track 48.1 -> 24.1 mm
- net Net-(J1-Pad35): track 24.1 -> 12.1 mm
- net Net-(J1-Pad23): track 24.4 -> 12.4 mm
- net Net-(J1-Pad19): track 24.1 -> 12.1 mm
- net Net-(J1-Pad13): track 24.1 -> 12.1 mm
- net Net-(J1-Pad7): track 24.1 -> 12.1 mm
- net Net-(J1-Pad5): track 24.1 -> 12.1 mm
- net Net-(J1-Pad33): track 24.1 -> 12.1 mm
- net Net-(J1-Pad3): track 24.1 -> 12.1 mm
- net Net-(J1-Pad29): track 24.1 -> 12.1 mm
- net Net-(J1-Pad15): track 24.1 -> 12.1 mm
- net Net-(J1-Pad11): track 24.1 -> 12.1 mm
- net Net-(J1-Pad37): track 24.1 -> 12.1 mm
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- added copper zone on F.Cu, net +3V3
- added copper zone on B.Cu, net GND
Other:
- board size 65 x 30 mm -> 65 x 18 mm
- board text added: "pi-bridge-2mm-1-1"
- board text removed: "pi-bridge-1-1"

Commit message: Release pi-bridge-2mm-1-2
Parts:
- removed the ? at (53.5, 63.5)
- removed the ? at (111.5, 63.5)
- added ?: , ice4pi:mount_hole, F.Cu at (53.5, 61.5)
- added ?: , ice4pi:mount_hole, F.Cu at (111.5, 61.5)
- moved J1 2.00 mm to (58.4, 62.8)
- moved svg2mod 1.00 mm to (99.0, 58.0)
Routing:
- net GND: track 96.6 -> 80.6 mm
- net +5V: track 24.1 -> 20.1 mm
- net +3V3: track 24.1 -> 20.1 mm
- net Net-(J1-Pad8): track 12.1 -> 10.1 mm
- net Net-(J1-Pad40): track 12.1 -> 10.1 mm
- net Net-(J1-Pad38): track 12.1 -> 10.1 mm
- net Net-(J1-Pad36): track 12.1 -> 10.1 mm
- net Net-(J1-Pad32): track 12.1 -> 10.1 mm
- net Net-(J1-Pad28): track 12.1 -> 10.1 mm
- net Net-(J1-Pad26): track 12.1 -> 10.1 mm
- net Net-(J1-Pad24): track 12.4 -> 10.4 mm
- net Net-(J1-Pad22): track 12.1 -> 10.1 mm
- net Net-(J1-Pad18): track 12.1 -> 10.1 mm
- net Net-(J1-Pad16): track 12.1 -> 10.1 mm
- net Net-(J1-Pad12): track 12.1 -> 10.1 mm
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Other:
- board size 65 x 18 mm -> 65 x 16 mm
- board text added: "pi-bridge-2mm-1-2"
- board text removed: "pi-bridge-2mm-1-1"
